File: Esp8266Interface/Esp8266Interface.kicad_pcb (KiCad board)
At the start: 2 copper layers, 23 parts, among them J1 ESP01, J2 Lx, J4 Lx, J5 Lx, J6 Lx, J7 Lx, Q1 2N7000, SW1 SW_Push, U1 LM1084-3.3, U2 PC817

Commit message: Circuit board
Parts:
- added J7: HV In, Connector_PinHeader_2.54mm:PinHeader_1x03_P2.54mm_Vertical, F.Cu at (126.0, 81.1)
- added R4: 47K, Resistor_THT:R_Axial_DIN0207_L6.3mm_D2.5mm_P2.54mm_Vertical, F.Cu at (133.5, 100.0)
- D2: footprint Diode_THT:D_DO-41_SOD81_P10.16mm_Horizontal -> Diode_THT:D_DO-41_SOD81_P5.08mm_Vertical_KathodeUp
- D3: footprint Diode_THT:D_DO-41_SOD81_P10.16mm_Horizontal -> Diode_THT:D_DO-41_SOD81_P3.81mm_Vertical_KathodeUp
- J2: value Lx -> In3
- J3: renamed from J7; value Lx -> In
- J4: value Lx -> Pin
- J5: value Lx -> Pout
- J6: value Lx -> Rly
- SW1: footprint Button_Switch_THT:SW_PUSH_6mm_H7.3mm -> Button_Switch_THT:SW_Tactile_Straight_KSL0Axx1LFTR
- moved C3 91.8 mm to (165.0, 113.0), turned to -90 degrees
- moved J2 70.3 mm to (175.0, 81.9), turned to 180 degrees
- moved J4 60.3 mm to (175.0, 98.8)
- moved J5 60.2 mm to (175.0, 107.9)
- moved C2 59.4 mm to (169.0, 81.9), turned to 180 degrees
- moved Q1 53.5 mm to (126.0, 108.2)
- moved C4 51.8 mm to (167.7, 98.9), turned to -90 degrees
- moved R3 42.7 mm to (133.9, 75.2)
- moved J6 39.1 mm to (135.5, 115.0), turned to -90 degrees
- moved SW1 39.0 mm to (149.6, 117.0), turned to 180 degrees
- moved C5 36.2 mm to (126.9, 91.0), turned to -90 degrees
- moved U2 26.0 mm to (149.9, 81.5)
- moved D3 25.0 mm to (137.4, 106.2), turned to 180 degrees
- moved D1 24.0 mm to (141.5, 88.4), turned to -90 degrees
- moved R1 22.8 mm to (141.4, 82.9), turned to 90 degrees
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Connections:
- J3 pad 1: Net-(J1-GPIO2) -> Net-(J1-GPIO0)
- J3 pad 2: Net-(J1-GPIO0) -> Net-(J1-GPIO2)
- R5 pad 2: Net-(J1-GPIO0) -> Net-(J1-GPIO2)
- R6 pad 2: Net-(J1-GPIO2) -> Net-(J1-GPIO0)
Routing:
- net GND: track 0.00 -> 234.6 mm
- net Net-(D3-K): track 0.00 -> 95.2 mm
- net +3.3V: track 0.00 -> 64.7 mm
- net Net-(D1-A): track 0.00 -> 46.1 mm
- net Net-(J1-Reset): track 0.00 -> 30.8 mm
- net Net-(J1-GPIO3): track 0.00 -> 29.8 mm
- net Net-(J1-GPIO2): track 0.00 -> 29.0 mm
- net Net-(J1-GPIO0): track 0.00 -> 25.9 mm
- net Net-(D1-K): track 0.00 -> 22.0 mm
- net Net-(J1-GPIO1): track 0.00 -> 18.1 mm
- net Net-(J7-Pin_2): track 0.00 -> 15.8 mm
- net Net-(Q1-G): track 0.00 -> 14.1 mm
- net Net-(D3-A): track 0.00 -> 13.2 mm
- net Net-(R1-Pad2): track 0.00 -> 8.95 mm
- net Net-(J7-Pin_3): track 0.00 -> 8.19 mm
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- added copper zone on F.Cu, net +3.3V
- added copper zone on B.Cu, net GND
Other:
- board outline added: 60 x 50 mm
