File: Esp8266Interface/Esp8266Interface.kicad_sch (KiCad schematic)
At the start: 25 parts, among them J1 ESP01, J2 Lx, J3 Screw_Terminal_01x03, Q1 2N7000, SW1 SW_Push, U1 LM1084-3.3, U2 PC817

Commit message: Circuit board
Parts:
- D2: footprint Diode_THT:D_DO-41_SOD81_P10.16mm_Horizontal -> Diode_THT:D_DO-41_SOD81_P5.08mm_Vertical_KathodeUp
- D3: footprint Diode_THT:D_DO-41_SOD81_P10.16mm_Horizontal -> Diode_THT:D_DO-41_SOD81_P3.81mm_Vertical_KathodeUp
- J2: value Lx -> Pin
- J2: value Lx -> Rly
- J2: value Lx -> Pout
- J2: value Lx -> In
- J2: value Lx -> In3
- J7: renamed from J3; value Screw_Terminal_01x03 -> HV In; footprint (none) -> Connector_PinHeader_2.54mm:PinHeader_1x03_P2.54mm_Vertical
- R4: footprint (none) -> Resistor_THT:R_Axial_DIN0207_L6.3mm_D2.5mm_P2.54mm_Vertical
- SW1: footprint Button_Switch_THT:SW_PUSH_6mm_H7.3mm -> Button_Switch_THT:SW_Tactile_Straight_KSL0Axx1LFTR
Connections:
- net at J2.1 (Pin_1), R6.2: now also J1.5 (GPIO0); no longer J1.3 (GPIO2)
- net at J2.2 (Pin_2), R5.2: now also J1.3 (GPIO2); no longer J1.5 (GPIO0)
Other:
- moved on the sheet: J2
